Commit message: asset fidelity stuff

File: data/lab_reconstruction/PRPL_lab/submodels/serial_abstract/urdf/serial_abstract.urdf (robot description, URDF)
Before this commit: robot serial_abstract, 60 links, 59 joints
Links:
- added link lab_in_progress_align_sink.149_link; visual mesh filename=../../../meshes/stl/lab_in_progress_align_sink.149.stl scale=1.00000 1.00000 1.00000
- added link lab_in_progress_align_sink.155_link; visual mesh filename=../../../meshes/stl/lab_in_progress_align_sink.155.stl scale=1.00000 1.00000 1.00000
- link Cabinet1.005_link: geometry 
Joints:
- added joint lab_in_progress_align_sink.149_link_joint: type revolute, parent lab_in_progress_align_sink.155_link, child lab_in_progress_align_sink.149_link, origin xyz=0.03723 0.25689 0.50505 rpy=-0.00000 -1.57080 0.00000, axis 0.00000 0.00000 1.00000, limit lower=0.00000 upper=1.50000 effort=0.00000 velocity=0.00000
- added joint sink: type fixed, parent Cabinet1.005_link, child lab_in_progress_align_sink.155_link, origin xyz=0.42532 -0.32433 0.39694 rpy=0.00000 0.00000 0.00000

File: data/lab_reconstruction/PRPL_lab/urdf/PRPL_lab.urdf (robot description, URDF)
Before this commit: robot PRPL_lab, 60 links, 59 joints
Links:
- added link lab_in_progress_align_sink.149_link; visual mesh filename=../meshes/stl/lab_in_progress_align_sink.149.stl scale=1.00000 1.00000 1.00000
- added link lab_in_progress_align_sink.155_link; visual mesh filename=../meshes/stl/lab_in_progress_align_sink.155.stl scale=1.00000 1.00000 1.00000
- link Baseboard2.001_link: geometry visual mesh filename=../meshes/stl/Baseboard2.001.stl scale=1.00000 1.00000 1.00000
- link Cabinet1.001_link: geometry visual mesh filename=../meshes/stl/Cabinet1.005.stl scale=1.00000 1.00000 1.00000
- link Cabinet1.002_link: geometry visual mesh filename=../meshes/stl/Cabinet1.002.stl scale=1.00000 1.00000 1.00000
- link Cabinet1.003_link: geometry visual mesh filename=../meshes/stl/Cabinet1.009.stl scale=1.00000 1.00000 1.00000
- link Cabinet1.004_link: geometry visual mesh filename=../meshes/stl/Cabinet1.003.stl scale=1.00000 1.00000 1.00000
- link Cabinet1.005_link: geometry 
- link Cabinet1.006_link: geometry visual mesh filename=../meshes/stl/Cabinet1.006.stl scale=1.00000 1.00000 1.00000
- link Cabinet1.007_link: geometry visual mesh filename=../meshes/stl/Cabinet1.001.stl scale=1.00000 1.00000 1.00000
- link Cabinet1_Door.001_link: geometry visual mesh filename=../meshes/stl/Cabinet1_Door.004.stl scale=1.00000 1.00000 1.00000
- link Cabinet1_Door.002_link: geometry visual mesh filename=../meshes/stl/Cabinet1_Door.002.stl scale=1.00000 1.00000 1.00000
- link Cabinet1_Door.003_link: geometry visual mesh filename=../meshes/stl/Cabinet1_Door.001.stl scale=1.00000 1.00000 1.00000
- link Cabinet1_Door.004_link: geometry visual mesh filename=../meshes/stl/Cabinet1_Door.005.stl scale=1.00000 1.00000 1.00000
- link Cabinet1_Door.005_link: geometry visual mesh filename=../meshes/stl/Cabinet1_Door.008.stl scale=1.00000 1.00000 1.00000
- link Cabinet1_Door.006_link: geometry visual mesh filename=../meshes/stl/Cabinet1_Door.006.stl scale=1.00000 1.00000 1.00000
- link Cabinet1_Door_link: geometry visual mesh filename=../meshes/stl/Cabinet1_Door.003.stl scale=1.00000 1.00000 1.00000
- link Cabinet1_link: geometry visual mesh filename=../meshes/stl/Cabinet1.004.stl scale=1.00000 1.00000 1.00000
- link Cabinet2_Door.001_link: geometry visual mesh filename=../meshes/stl/Cabinet2_Door.003.stl scale=1.00000 1.00000 1.00000
- link Cabinet2_Door.002_link: geometry visual mesh filename=../meshes/stl/Cabinet2_Door.001.stl scale=1.00000 1.00000 1.00000
- link Cabinet2_Door.003_link: geometry visual mesh filename=../meshes/stl/Cabinet2_Door.005.stl scale=1.00000 1.00000 1.00000
- link Cabinet2_Door.004_link: geometry visual mesh filename=../meshes/stl/Cabinet2_Door.007.stl scale=1.00000 1.00000 1.00000
- link Cabinet2_Door.005_link: geometry visual mesh filename=../meshes/stl/Cabinet2_Door.004.stl scale=1.00000 1.00000 1.00000
- link Cabinet2_Door_link: geometry visual mesh filename=../meshes/stl/Cabinet2_Door.002.stl scale=1.00000 1.00000 1.00000
- link Countertop1.001_link: geometry visual mesh filename=../meshes/stl/Countertop1.stl scale=1.00000 1.00000 1.00000
- link Countertop1_link: geometry visual mesh filename=../meshes/stl/Countertop1.002.stl scale=1.00000 1.00000 1.00000; visual mesh filename=../meshes/stl/base.stl scale=1.00000 1.00000 1.00000
- link Drawer.001_link: geometry visual mesh filename=../meshes/stl/Drawer.004.stl scale=1.00000 1.00000 1.00000
- link Drawer.002_link: geometry visual mesh filename=../meshes/stl/Drawer.005.stl scale=1.00000 1.00000 1.00000
- link Drawer.003_link: geometry visual mesh filename=../meshes/stl/Drawer.012.stl scale=1.00000 1.00000 1.00000
- link Drawer.004_link: geometry visual mesh filename=../meshes/stl/Drawer.013.stl scale=1.00000 1.00000 1.00000
- link Drawer.005_link: geometry visual mesh filename=../meshes/stl/Drawer.014.stl scale=1.00000 1.00000 1.00000
- link Drawer_link: geometry visual mesh filename=../meshes/stl/Drawer.003.stl scale=1.00000 1.00000 1.00000
- link Handle.001_link: geometry visual mesh filename=../meshes/stl/Handle.004.stl scale=1.00000 1.00000 1.00000
- link Handle.002_link: geometry visual mesh filename=../meshes/stl/Handle.005.stl scale=1.00000 1.00000 1.00000
- link Handle.003_link: geometry visual mesh filename=../meshes/stl/Handle.002.stl scale=1.00000 1.00000 1.00000
- link Handle.004_link: geometry visual mesh filename=../meshes/stl/Handle.003.stl scale=1.00000 1.00000 1.00000
- link Handle.005_link: geometry visual mesh filename=../meshes/stl/Handle.006.stl scale=1.00000 1.00000 1.00000
- link Handle.006_link: geometry visual mesh filename=../meshes/stl/Handle.007.stl scale=1.00000 1.00000 1.00000
- link Handle.007_link: geometry visual mesh filename=../meshes/stl/Handle.011.stl scale=1.00000 1.00000 1.00000
- link Handle.008_link: geometry visual mesh filename=../meshes/stl/Handle.012.stl scale=1.00000 1.00000 1.00000
- link Handle.012_link: geometry visual mesh filename=../meshes/stl/Handle.009.stl scale=1.00000 1.00000 1.00000
- link Handle.013_link: geometry visual mesh filename=../meshes/stl/Handle.010.stl scale=1.00000 1.00000 1.00000
- link Handle_link: geometry visual mesh filename=../meshes/stl/Handle.008.stl scale=1.00000 1.00000 1.00000
- link base.001_link: geometry visual mesh filename=../meshes/stl/base.002.stl scale=1.00000 1.00000 1.00000
- link base.002_link: geometry visual mesh filename=../meshes/stl/base.001.stl scale=1.00000 1.00000 1.00000
- link door_0.001_link: geometry visual mesh filename=../meshes/stl/door_0.002.stl scale=1.00000 1.00000 1.00000
- link door_0.002_link: geometry visual mesh filename=../meshes/stl/door_0.001.stl scale=1.00000 1.00000 1.00000
- link door_0_link: geometry visual mesh filename=../meshes/stl/door_0.stl scale=1.00000 1.00000 1.00000
- link door_1_link: geometry visual mesh filename=../meshes/stl/door_1.001.stl scale=1.00000 1.00000 1.00000
- link door_2_link: geometry visual mesh filename=../meshes/stl/door_2.001.stl scale=1.00000 1.00000 1.00000
- link door_3_link: geometry visual mesh filename=../meshes/stl/door_3.001.stl scale=1.00000 1.00000 1.00000
- link new_link: geometry visual mesh filename=../meshes/stl/stoveCube.stl scale=1.00000 1.00000 1.00000
- link stovestove-door.002_link: geometry visual mesh filename=../meshes/stl/stovestove-door.004.stl scale=1.00000 1.00000 1.00000
- link stovestove-knob.001_link: geometry visual mesh filename=../meshes/stl/stovestove-knob.001.stl scale=1.00000 1.00000 1.00000
- link stovestove-knob.002_link: geometry visual mesh filename=../meshes/stl/stovestove-knob.002.stl scale=1.00000 1.00000 1.00000
- link stovestove-knob.003_link: geometry visual mesh filename=../meshes/stl/stovestove-knob.003.stl scale=1.00000 1.00000 1.00000
- link stovestove-knob.004_link: geometry visual mesh filename=../meshes/stl/stovestove-knob.004.stl scale=1.00000 1.00000 1.00000
- link stovestove-knob_link: geometry visual mesh filename=../meshes/stl/stovestove-knob.stl scale=1.00000 1.00000 1.00000
Joints:
- added joint lab_in_progress_align_sink.149_link_joint: type revolute, parent lab_in_progress_align_sink.155_link, child lab_in_progress_align_sink.149_link, origin xyz=0.03723 0.25689 0.50505 rpy=-0.00000 -1.57080 0.00000, axis 0.00000 0.00000 1.00000, limit lower=0.00000 upper=1.50000 effort=0.00000 velocity=0.00000
- added joint sink: type fixed, parent Cabinet1.005_link, child lab_in_progress_align_sink.155_link, origin xyz=0.42532 -0.32433 0.39694 rpy=0.00000 0.00000 0.00000

File: data/output/urdf_test/name.urdf (robot description, URDF)
Before this commit: robot articulated_object, 3 links, 2 joints
Links:
- removed link door_1
Joints:
- removed joint joint_1
- joint joint_0: origin xyz=3.98423545 0.67850360 1.11890409 rpy=0 0 0 -> xyz=0.45650975 0.20805626 0.06646188 rpy=0 0 0
