Commit message: updated UI

File: data/output/urdf_test/name.urdf (robot description, URDF)
Before this commit: robot articulated_object, 2 links, 1 joints
Joints:
- joint joint1: axis 0.99619470 -0.08715574 0.00000000 -> 0.99666593 -0.08159061 0.00000000; limit lower=0.0 upper=0.17453292519943295 effort=100.0 velocity=1.0 -> lower=0.0 upper=0.5235987755982988 effort=100.0 velocity=1.0; origin xyz=-1.24774950 -1.09099688 -0.30609245 rpy=0 0 0 -> xyz=-1.41229273 -1.06644984 -0.29216917 rpy=0 0 0

Commit message: capping works, watertight cap creation

File: data/output/urdf_test/name.urdf (robot description, URDF)
Before this commit: robot articulated_object, 2 links, 1 joints
Joints:
- joint joint1: axis 0.99666593 -0.08159061 0.00000000 -> 0.99871936 -0.05059294 0.00000000; limit lower=0.0 upper=0.5235987755982988 effort=100.0 velocity=1.0 -> lower=-1.5707963267948966 upper=1.5707963267948966 effort=100.0 velocity=1.0; origin xyz=-1.41229273 -1.06644984 -0.29216917 rpy=0 0 0 -> xyz=-1.29249782 -1.08654138 -0.29115028 rpy=0 0 0

Commit message: capping doesnt work but door does but im so tired and i cant do this anymore:

File: data/output/urdf_test/name.urdf (robot description, URDF)
Before this commit: robot articulated_object, 2 links, 1 joints
Joints:
- joint joint1: axis 0.99871936 -0.05059294 0.00000000 -> 0.00000000 1.00000000 0.00000000; limit lower=-1.5707963267948966 upper=1.5707963267948966 effort=100.0 velocity=1.0 -> lower=0.0 upper=0.7853981633974483 effort=100.0 velocity=1.0; origin xyz=-1.29249782 -1.08654138 -0.29115028 rpy=0 0 0 -> xyz=0.10403955 -0.52233721 0.20490544 rpy=0 0 0

Commit message: committing before i mess up cuboid by knife algo experimentation

File: data/output/urdf_test/name.urdf (robot description, URDF)
Before this commit: robot articulated_object, 2 links, 1 joints
Joints:
- joint joint1: axis 0.00000000 1.00000000 0.00000000 -> 0.00000000 0.00000000 1.00000000; limit lower=0.0 upper=0.7853981633974483 effort=100.0 velocity=1.0 -> lower=0.0 upper=0.3490658503988659 effort=100.0 velocity=1.0; origin xyz=0.10403955 -0.52233721 0.20490544 rpy=0 0 0 -> xyz=274.97239110 -110.81053353 1351.72545322 rpy=0 0 0

Commit message: Door with thickness, projects largest boundary to back cuboidal plane

File: data/output/urdf_test/name.urdf (robot description, URDF)
Before this commit: robot articulated_object, 2 links, 1 joints
Joints:
- joint joint1: origin xyz=274.97239110 -110.81053353 1351.72545322 rpy=0 0 0 -> xyz=261.48991930 -102.32125482 1357.70861164 rpy=0 0 0

Commit message: door

File: data/output/urdf_test/name.urdf (robot description, URDF)
Before this commit: robot articulated_object, 2 links, 1 joints
Joints:
- joint joint1: axis 0.00000000 0.00000000 1.00000000 -> 1.00000000 0.00000000 0.00000000; limit lower=0.0 upper=0.3490658503988659 effort=100.0 velocity=1.0 -> lower=0.0 upper=0.6981317007977318 effort=100.0 velocity=1.0; origin xyz=261.48991930 -102.32125482 1357.70861164 rpy=0 0 0 -> xyz=-34.87687583 -23.09956412 22.05954968 rpy=0 0 0

Commit message: multiple door selection possible, cleanup for disconnected components needed

File: data/output/urdf_test/name.urdf (robot description, URDF)
Before this commit: robot articulated_object, 2 links, 1 joints
Links:
- removed link child
- removed link parent
- added link base; visual mesh filename=base.stl
- added link door_0; visual mesh filename=door_0.stl
- added link door_1; visual mesh filename=door_1.stl
Joints:
- removed joint joint1
- added joint joint_0: type revolute, parent base, child door_0, origin xyz=0.44930416 0.20419391 0.06589369 rpy=0 0 0, axis 0.00000000 0.00000000 1.00000000, limit lower=0.0 upper=1.5707963267948966 effort=100.0 velocity=1.0
- added joint joint_1: type revolute, parent base, child door_1, origin xyz=-0.20118648 -0.45544330 1.40710630 rpy=0 0 0, axis 0.00000000 0.00000000 -1.00000000, limit lower=0.0 upper=1.5707963267948966 effort=100.0 velocity=1.0

Commit message: can save split meshes

File: data/output/urdf_test/name.urdf (robot description, URDF)
Before this commit: robot articulated_object, 3 links, 2 joints
Links:
- removed link door_1
Joints:
- removed joint joint_1
- joint joint_0: axis 0.00000000 0.00000000 1.00000000 -> 0.08524845 0.94817156 0.30611009; limit lower=0.0 upper=1.5707963267948966 effort=100.0 velocity=1.0 -> lower=-1.2189379495928399 upper=1.5707963267948966 effort=100.0 velocity=1.0; origin xyz=0.44930416 0.20419391 0.06589369 rpy=0 0 0 -> xyz=2.79114381 -0.74324778 -0.03488319 rpy=0 0 0

Commit message: PRPL URDF via blender, tool with cylindrical selection

File: data/output/urdf_test/name.urdf (robot description, URDF)
Before this commit: robot articulated_object, 2 links, 1 joints
Links:
- added link door_1; visual mesh filename=door_1.stl
Joints:
- added joint joint_1: type continuous, parent base, child door_1, origin xyz=3.94985473 0.60714909 1.03227347 rpy=0 0 0, axis 0.00000000 -1.00000000 0.00000000
- joint joint_0: axis 0.08524845 0.94817156 0.30611009 -> 0.00000000 0.00000000 1.00000000; limit lower=-1.2189379495928399 upper=1.5707963267948966 effort=100.0 velocity=1.0 -> lower=0.0 upper=1.3089969389957472 effort=100.0 velocity=1.0; origin xyz=2.79114381 -0.74324778 -0.03488319 rpy=0 0 0 -> xyz=3.98423545 0.67850360 1.11890409 rpy=0 0 0

Commit message: fixed camera reset bug

File: data/output/urdf_test/name.urdf (robot description, URDF)
Before this commit: robot articulated_object, 2 links, 1 joints
Links:
- added link door_1; visual mesh filename=door_1.stl
- added link door_2; visual mesh filename=door_2.stl
- added link door_3; visual mesh filename=door_3.stl
- added link door_4; visual mesh filename=door_4.stl
Joints:
- added joint joint_1: type revolute, parent base, child door_1, origin xyz=1.25957137 3.44370797 2.18808459 rpy=0 0 0, axis 0.00000000 0.00000000 -1.00000000, limit lower=0.0 upper=1.3089969389957472 effort=100.0 velocity=1.0
- added joint joint_2: type revolute, parent base, child door_2, origin xyz=1.94390429 2.93917422 1.30240181 rpy=0 0 0, axis 0.00000000 0.00000000 1.00000000, limit lower=0.0 upper=1.3089969389957472 effort=100.0 velocity=1.0
- added joint joint_3: type revolute, parent base, child door_3, origin xyz=1.24660140 0.71035769 -0.24380492 rpy=0 0 0, axis 0.00000000 0.00000000 1.00000000, limit lower=0.0 upper=1.3089969389957472 effort=100.0 velocity=1.0
- added joint joint_4: type revolute, parent base, child door_4, origin xyz=1.24778859 0.71191046 0.82024347 rpy=0 0 0, axis 0.00000000 0.00000000 1.00000000, limit lower=0.0 upper=1.3089969389957472 effort=100.0 velocity=1.0
- joint joint_0: axis 0.00000000 0.00000000 1.00000000 -> 0.80489380 -0.59341889 0.00000000; origin xyz=0.45650975 0.20805626 0.06646188 rpy=0 0 0 -> xyz=0.78050875 3.37366374 0.06218131 rpy=0 0 0

Commit message: kitchen urdf with cabinet selection

File: data/output/urdf_test/name.urdf (robot description, URDF)
Before this commit: robot articulated_object, 6 links, 5 joints
Links:
- added link door_5; visual mesh filename=door_5.stl
- added link door_6; visual mesh filename=door_6.stl
Joints:
- added joint joint_5: type revolute, parent base, child door_5, origin xyz=3.00276059 2.03885339 1.47078759 rpy=0 0 0, axis 0.00000000 0.00000000 -1.00000000, limit lower=0.0 upper=1.3089969389957472 effort=100.0 velocity=1.0
- added joint joint_6: type revolute, parent base, child door_6, origin xyz=2.48276147 1.35921457 1.06113375 rpy=0 0 0, axis 0.00000000 0.00000000 1.00000000, limit lower=0.0 upper=1.3089969389957472 effort=100.0 velocity=1.0
- joint joint_0: axis 0.80489380 -0.59341889 0.00000000 -> 0.80942715 -0.58722031 0.00000000; origin xyz=0.78050875 3.37366374 0.06218131 rpy=0 0 0 -> xyz=0.72587861 3.34588627 0.06155931 rpy=0 0 0
- joint joint_1: origin xyz=1.25957137 3.44370797 2.18808459 rpy=0 0 0 -> xyz=1.24694521 3.42703056 2.22879387 rpy=0 0 0
- joint joint_2: origin xyz=1.94390429 2.93917422 1.30240181 rpy=0 0 0 -> xyz=1.95692207 2.91195909 1.32162002 rpy=0 0 0
- joint joint_3: origin xyz=1.24660140 0.71035769 -0.24380492 rpy=0 0 0 -> xyz=1.23535171 0.69724409 -0.25977094 rpy=0 0 0
- joint joint_4: origin xyz=1.24778859 0.71191046 0.82024347 rpy=0 0 0 -> xyz=1.23535171 0.69724409 0.87685460 rpy=0 0 0

Commit message: fixed plane bounds

File: data/output/urdf_test/name.urdf (robot description, URDF)
Before this commit: robot articulated_object, 8 links, 7 joints
Links:
- removed link door_1
- removed link door_2
- removed link door_3
- removed link door_4
- removed link door_5
- removed link door_6
Joints:
- removed joint joint_1
- removed joint joint_2
- removed joint joint_3
- removed joint joint_4
- removed joint joint_5
- removed joint joint_6
- joint joint_0: axis 0.80942715 -0.58722031 0.00000000 -> 0.00000000 0.00000000 -1.00000000; origin xyz=0.72587861 3.34588627 0.06155931 rpy=0 0 0 -> xyz=1.11697522 -0.71617644 1.83723763 rpy=0 0 0

Commit message: drawer

File: data/output/urdf_test/name.urdf (robot description, URDF)
Before this commit: robot articulated_object, 2 links, 1 joints
Links:
- added link door_1; visual mesh filename=door_1.stl
Joints:
- added joint joint_1: type prismatic, parent base, child door_1, origin xyz=-4.78927802 -1.88207018 5.91022464 rpy=0 0 0, axis -0.00000000 1.00000000 0.00000000, limit lower=0.0 upper=7.347 effort=100.0 velocity=1.0
- joint joint_0: axis 0.00000000 0.00000000 -1.00000000 -> -0.00000000 1.00000000 0.00000000; limit lower=0.0 upper=1.3089969389957472 effort=100.0 velocity=1.0 -> lower=0.0 upper=7.347 effort=100.0 velocity=1.0; origin xyz=1.11697522 -0.71617644 1.83723763 rpy=0 0 0 -> xyz=-4.81574610 -1.88207018 3.97006284 rpy=0 0 0; type revolute -> prismatic

Commit message: before final code cleanup

File: data/output/urdf_test/name.urdf (robot description, URDF)
Before this commit: robot articulated_object, 3 links, 2 joints
Joints:
- joint joint_0: axis -0.00000000 1.00000000 0.00000000 -> 0.00000000 1.00000000 0.00000000; limit lower=0.0 upper=7.347 effort=100.0 velocity=1.0 -> lower=0.0 upper=7.229 effort=100.0 velocity=1.0; origin xyz=-4.81574610 -1.88207018 3.97006284 rpy=0 0 0 -> xyz=-4.81113793 -1.09300743 5.83019529 rpy=0 0 0
- joint joint_1: axis -0.00000000 1.00000000 0.00000000 -> 0.00000000 0.00000000 1.00000000; limit lower=0.0 upper=7.347 effort=100.0 velocity=1.0 -> lower=0.0 upper=0.12616985162667008 effort=100.0 velocity=1.0; origin xyz=-4.78927802 -1.88207018 5.91022464 rpy=0 0 0 -> xyz=-4.77848371 2.38260326 7.44879069 rpy=0 0 0; type prismatic -> revolute
